File: USBBoost.sch (EAGLE design)
At the start: 27 parts, among them IC1 RT9276, J2 3.75V, J3 2.33V, J4 1.17V, J5 Status, X1 USB_

Commit message: v1.1 release
Parts:
- removed B1: 2P-JST-PTH, freetronics-jon:FREETRONICS-LUKE_2P-JST-TH-RAPTH
- removed J4: 1.17V, freetronics-luke:SJ
- removed J5: Status, freetronics-master-v1:M02PTH
- removed X1: USB_, freetronics-master-v1:USB_
- added H1: 2P-JST-PTH, freetronics-jon:2P-JST-TH-RAPTH
- added H2: (no value), freetronics-master-v1.1:M02PTH
- added H3: USB, freetronics-master-v1:USB_
- added H4: Status, freetronics-master-v1:M02PTH
- added J1: 3.75V, freetronics-jon:SJCN
- C1: value 10uF ceramic -> 10uF ceramic 10V 0805
- C2: value 22uF -> 22uF 10V Ceramic 1206
- F1: value 500mA PTC -> 500mA PTC 1812
- J2: value 3.75V -> 2.33V
- J3: value 2.33V -> 1.17V
- L1: value 7.4uH -> 7.4uH CDRH
- LED1: value Power -> BLUE 0603
- LED2: value Low Batt -> RED 0603
- R1: value 130K -> 130K 0603
- R10: value 1K -> 75K 0603
- R11: value 75K -> 49K9 0603
- R12: value 49K9 -> 49K9 0603
- R13: value 75K -> 20K 0603
- R14: value 49K9 -> 20K0 1% 0603
- R2: value 20K -> 73K2 0603
- R3: value 73K2 -> 26K7 0603
- R4: value 26K7 -> 180K 1% 0603
- R5: value 180K -> 10K 0603
- R6: value 20K0 -> 10K 0603
- R7: value 10K -> 2K2 0603
- R8: value 10K -> 1K 0603
- R9: value 2K2 -> 75K 0603
Connections:
- removed net N$12 (its old number): J4.1, R4.2
- new net N$11: J2.1, R2.2
- net !LBO: now also H4.2, R6.2; no longer J5.2, R8.2
- net !PGOOD: now also H4.1, R5.2; no longer J5.1, R7.2
- net FB: now also R14.2, R4.2; no longer R5.2, R6.2
- net GND: now also H1.NEG, H2.1, H3.GND, R11.2, R13.1, R14.1; no longer B1.NEG, R14.2, R2.1, R6.1, X1.GND
- net LBI: now also R13.2, R2.1; no longer R2.2, R4.1
- net N$10: now also H3.D+, R10.2, R12.1; no longer R13.2, R14.1, X1.D+
- net N$15: now also R8.2; no longer R10.2
- net N$5: now also J1.1; no longer J2.1
- net N$7: now also H3.D-, R11.1, R9.2; no longer R11.2, R12.1, X1.D-
- net N$8: now also R7.2; no longer R9.2
- net N$9: now also H3.VBUS; no longer X1.VBUS
- net VBAT: now also H1.POS, H2.2, J1.2; no longer B1.POS, J4.2
- net VOUT: now also R4.1, R6.1; no longer R11.1, R13.1
Other:
- note added: "(C)2013 Freetronics Pty Ltd: www.freetronics.com"
- note added: "H3"
- note added: "Jumpers J1, J2, and J3 change the input voltage to the internal low-battery comparator output."
- note added: "Low Batt"
- note added: "Power"
- note added: "V1.1 (2013-05-06)"
- note removed: "(C)2012 Freetronics Pty Ltd: www.freetronics.com"
- note removed: "0603"
- note removed: "1%"
- note removed: "10V"
- note removed: "1812"
- note removed: "Blue"
- note removed: "Bridge across J2 after other routing"
- note removed: "CDRH"
- note removed: "Jumpers J2, J3 and J4 change the input voltage to the internal low-battery comparator output."
- note removed: "Red"
- note removed: "V1.0 (13-06-2012)"
- moved on the sheet: F1, J2, J3, LED2, R10, R11, R12, R13, R14, R2, R3, R4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
